File: Board1 - kicad/Tic_Tac-Toe Analogue.sch (KiCad schematic (older format))
At the start: 43 parts, among them CON1 BARREL_JACK, P1 CONN_01X12, P2 CONN_02X10, SW1 SW_PUSH_4, SW10 SW_PUSH_4, SW11 SWITCH_INV, SW2 SW_PUSH_4, SW3 SW_PUSH_4, SW4 SW_PUSH_4, SW5 SW_PUSH_4, SW6 SW_PUSH_4, SW7 SW_PUSH_4, SW8 SW_PUSH_4, SW9 SW_PUSH_4

Commit message: Work on Top Board
Parts:
- D1, D10, D11, D12, D13, D14, D15, D16, D17, D18, D19, D2, D20, D3, D4, D5, D6, D7, D8, D9: footprint LEDs:LED-5MM -> LEDs:LED_D5.0mm
- R1, R2, R3, R4, R5, R6: footprint Resistors_ThroughHole:Resistor_Horizontal_RM7mm -> Resistors_ThroughHole:R_Axial_DIN0207_L6.3mm_D2.5mm_P10.16mm_Horizontal
Connections:
- net GND: no longer R1.1, R2.1, RR1.9, SW1.2, SW10.2, SW2.2, SW3.2, SW4.2, SW5.2, SW6.2, SW7.2, SW8.2, SW9.2
- new net: R1.1, R2.1, RR1.9, SW1.2, SW10.2, SW2.2, SW3.2, SW4.2, SW5.2, SW6.2, SW7.2, SW8.2, SW9.2
Changed lines of the file:
@@
 F 0 "D2" H 2550 5300 50  0000 C CNN
 F 1 "LED" H 2550 5100 50  0000 C CNN
-F 2 "LEDs:LED-5MM" H 2550 5200 50  0001 C CNN
+F 2 "LEDs:LED_D5.0mm" H 2550 5200 50  0001 C CNN
 F 3 "" H 2550 5200 50  0000 C CNN
 	1    2550 5200
@@
 F 0 "D5" H 2550 7400 50  0000 C CNN
 F 1 "LED" H 2550 7200 50  0000 C CNN
-F 2 "LEDs:LED-5MM" H 2550 7300 50  0001 C CNN
+F 2 "LEDs:LED_D5.0mm" H 2550 7300 50  0001 C CNN
 F 3 "" H 2550 7300 50  0000 C CNN
 	1    2550 7300
@@
 F 0 "D12" H 4000 5300 50  0000 C CNN
 F 1 "LED" H 4000 5100 50  0000 C CNN
-F 2 "LEDs:LED-5MM" H 4000 5200 50  0001 C CNN
+F 2 "LEDs:LED_D5.0mm" H 4000 5200 50  0001 C CNN
 F 3 "" H 4000 5200 50  0000 C CNN
 	1    4000 5200
@@
 F 0 "D3" H 2550 5900 50  0000 C CNN
 F 1 "LED" H 2550 5700 50  0000 C CNN
-F 2 "LEDs:LED-5MM" H 2550 5800 50  0001 C CNN
+F 2 "LEDs:LED_D5.0mm" H 2550 5800 50  0001 C CNN
 F 3 "" H 2550 5800 50  0000 C CNN
 	1    2550 5800
@@
 F 0 "D15" H 4000 7400 50  0000 C CNN
 F 1 "LED" H 4000 7200 50  0000 C CNN
-F 2 "LEDs:LED-5MM" H 4000 7300 50  0001 C CNN
+F 2 "LEDs:LED_D5.0mm" H 4000 7300 50  0001 C CNN
 F 3 "" H 4000 7300 50  0000 C CNN
 	1    4000 7300
@@
 F 0 "D13" H 4000 5900 50  0000 C CNN
 F 1 "LED" H 4000 5700 50  0000 C CNN
-F 2 "LEDs:LED-5MM" H 4000 5800 50  0001 C CNN
+F 2 "LEDs:LED_D5.0mm" H 4000 5800 50  0001 C CNN
 F 3 "" H 4000 5800 50  0000 C CNN
 	1    4000 5800
@@
 F 0 "D1" H 2550 4750 50  0000 C CNN
 F 1 "LED" H 2550 4550 50  0000 C CNN
-F 2 "LEDs:LED-5MM" H 2550 4650 50  0001 C CNN
+F 2 "LEDs:LED_D5.0mm" H 2550 4650 50  0001 C CNN
 F 3 "" H 2550 4650 50  0000 C CNN
 	1    2550 4650
@@
 F 0 "D4" H 2550 6600 50  0000 C CNN
 F 1 "LED" H 2550 6400 50  0000 C CNN
-F 2 "LEDs:LED-5MM" H 2550 6500 50  0001 C CNN
+F 2 "LEDs:LED_D5.0mm" H 2550 6500 50  0001 C CNN
 F 3 "" H 2550 6500 50  0000 C CNN
 	1    2550 6500
@@
 F 0 "D11" H 4000 4750 50  0000 C CNN
 F 1 "LED" H 4000 4550 50  0000 C CNN
-F 2 "LEDs:LED-5MM" H 4000 4650 50  0001 C CNN
+F 2 "LEDs:LED_D5.0mm" H 4000 4650 50  0001 C CNN
 F 3 "" H 4000 4650 50  0000 C CNN
 	1    4000 4650
@@
 F 0 "D7" H 3250 5300 50  0000 C CNN
 F 1 "LED" V 3250 5100 50  0000 C CNN
-F 2 "LEDs:LED-5MM" H 3250 5200 50  0001 C CNN
+F 2 "LEDs:LED_D5.0mm" H 3250 5200 50  0001 C CNN
 F 3 "" H 3250 5200 50  0000 C CNN
 	1    3250 5200
@@
 F 0 "D14" H 4000 6600 50  0000 C CNN
 F 1 "LED" H 4000 6400 50  0000 C CNN
-F 2 "LEDs:LED-5MM" H 4000 6500 50  0001 C CNN
+F 2 "LEDs:LED_D5.0mm" H 4000 6500 50  0001 C CNN
 F 3 "" H 4000 6500 50  0000 C CNN
 	1    4000 6500
@@
 F 0 "D17" H 4750 5300 50  0000 C CNN
 F 1 "LED" H 4750 5100 50  0000 C CNN
-F 2 "LEDs:LED-5MM" H 4750 5200 50  0001 C CNN
+F 2 "LEDs:LED_D5.0mm" H 4750 5200 50  0001 C CNN
 F 3 "" H 4750 5200 50  0000 C CNN
 	1    4750 5200
@@
 F 0 "D8" H 3250 5900 50  0000 C CNN
 F 1 "LED" H 3250 5700 50  0000 C CNN
-F 2 "LEDs:LED-5MM" H 3250 5800 50  0001 C CNN
+F 2 "LEDs:LED_D5.0mm" H 3250 5800 50  0001 C CNN
 F 3 "" H 3250 5800 50  0000 C CNN
 	1    3250 5800
@@
 F 0 "D20" H 4750 7400 50  0000 C CNN
 F 1 "LED" H 4750 7200 50  0000 C CNN
-F 2 "LEDs:LED-5MM" H 4750 7300 50  0001 C CNN
+F 2 "LEDs:LED_D5.0mm" H 4750 7300 50  0001 C CNN
 F 3 "" H 4750 7300 50  0000 C CNN
 	1    4750 7300
@@
 F 0 "D18" H 4750 5900 50  0000 C CNN
 F 1 "LED" H 4750 5700 50  0000 C CNN
-F 2 "LEDs:LED-5MM" H 4750 5800 50  0001 C CNN
+F 2 "LEDs:LED_D5.0mm" H 4750 5800 50  0001 C CNN
 F 3 "" H 4750 5800 50  0000 C CNN
 	1    4750 5800
@@
 F 0 "D6" H 3250 4750 50  0000 C CNN
 F 1 "LED" H 3250 4550 50  0000 C CNN
-F 2 "LEDs:LED-5MM" H 3250 4650 50  0001 C CNN
+F 2 "LEDs:LED_D5.0mm" H 3250 4650 50  0001 C CNN
 F 3 "" H 3250 4650 50  0000 C CNN
 	1    3250 4650
@@
 F 0 "D9" V 3250 6600 50  0000 C CNN
 F 1 "LED" H 3250 6400 50  0000 C CNN
-F 2 "LEDs:LED-5MM" H 3250 6500 50  0001 C CNN
+F 2 "LEDs:LED_D5.0mm" H 3250 6500 50  0001 C CNN
 F 3 "" H 3250 6500 50  0000 C CNN
 	1    3250 6500
@@
 F 0 "D16" H 4750 4750 50  0000 C CNN
 F 1 "LED" H 4750 4550 50  0000 C CNN
-F 2 "LEDs:LED-5MM" H 4750 4650 50  0001 C CNN
+F 2 "LEDs:LED_D5.0mm" H 4750 4650 50  0001 C CNN
 F 3 "" H 4750 4650 50  0000 C CNN
 	1    4750 4650
@@
 F 0 "D10" H 3250 7400 50  0000 C CNN
 F 1 "LED" H 3250 7200 50  0000 C CNN
-F 2 "LEDs:LED-5MM" H 3250 7300 50  0001 C CNN
+F 2 "LEDs:LED_D5.0mm" H 3250 7300 50  0001 C CNN
 F 3 "" H 3250 7300 50  0000 C CNN
 	1    3250 7300
@@
 F 0 "D19" H 4750 6600 50  0000 C CNN
 F 1 "LED" H 4750 6400 50  0000 C CNN
-F 2 "LEDs:LED-5MM" H 4750 6500 50  0001 C CNN
+F 2 "LEDs:LED_D5.0mm" H 4750 6500 50  0001 C CNN
 F 3 "" H 4750 6500 50  0000 C CNN
 	1    4750 6500
@@
 F 0 "R1" V 2830 3250 50  0000 C CNN
 F 1 "10k" V 2750 3250 50  0000 C CNN
-F 2 "Resistors_ThroughHole:Resistor_Horizontal_RM7mm" V 2680 3250 50  0001 C CNN
+F 2 "Resistors_ThroughHole:R_Axial_DIN0207_L6.3mm_D2.5mm_P10.16mm_Horizontal" V 2680 3250 50  0001 C CNN
 F 3 "" H 2750 3250 50  0000 C CNN
 	1    2750 3250
@@
 F 0 "R4" V 6030 3900 50  0000 C CNN
 F 1 "200R" V 5950 3900 50  0000 C CNN
-F 2 "Resistors_ThroughHole:Resistor_Horizontal_RM7mm" V 5880 3900 50  0001 C CNN
+F 2 "Resistors_ThroughHole:R_Axial_DIN0207_L6.3mm_D2.5mm_P10.16mm_Horizontal" V 5880 3900 50  0001 C CNN
 F 3 "" H 5950 3900 50  0000 C CNN
 	1    5950 3900
@@
 F 0 "R5" V 6030 4100 50  0000 C CNN
 F 1 "200R" V 5950 4100 50  0000 C CNN
-F 2 "Resistors_ThroughHole:Resistor_Horizontal_RM7mm" V 5880 4100 50  0001 C CNN
+F 2 "Resistors_ThroughHole:R_Axial_DIN0207_L6.3mm_D2.5mm_P10.16mm_Horizontal" V 5880 4100 50  0001 C CNN
 F 3 "" H 5950 4100 50  0000 C CNN
 	1    5950 4100
@@
 F 0 "R2" V 5780 1100 50  0000 C CNN
 F 1 "10k" V 5700 1100 50  0000 C CNN
-F 2 "Resistors_ThroughHole:Resistor_Horizontal_RM7mm" V 5630 1100 50  0001 C CNN
+F 2 "Resistors_ThroughHole:R_Axial_DIN0207_L6.3mm_D2.5mm_P10.16mm_Horizontal" V 5630 1100 50  0001 C CNN
 F 3 "" H 5700 1100 50  0000 C CNN
 	1    5700 1100
@@
 	1    0    0    -1
 $EndComp
-$Comp
-L GND #PWR03
-U 1 1 5839B3ED
-P 6050 2950
-F 0 "#PWR03" H 6050 2700 50  0001 C CNN
-F 1 "GND" H 6050 2800 50  0000 C CNN
-F 2 "" H 6050 2950 50  0000 C CNN
-F 3 "" H 6050 2950 50  0000 C CNN
-	1    6050 2950
-	0    -1   -1   0
-$EndComp
 Wire Wire Line
 	2950 6500 3050 6500
@@
 F 0 "R3" V 6030 3700 50  0000 C CNN
 F 1 "200R" V 5950 3700 50  0000 C CNN
-F 2 "Resistors_ThroughHole:Resistor_Horizontal_RM7mm" V 5880 3700 50  0001 C CNN
+F 2 "Resistors_ThroughHole:R_Axial_DIN0207_L6.3mm_D2.5mm_P10.16mm_Horizontal" V 5880 3700 50  0001 C CNN
 F 3 "" H 5950 3700 50  0000 C CNN
 	1    5950 3700
@@
 F 0 "R6" V 6030 4300 50  0000 C CNN
 F 1 "200R" V 5950 4300 50  0000 C CNN
-F 2 "Resistors_ThroughHole:Resistor_Horizontal_RM7mm" V 5880 4300 50  0001 C CNN
+F 2 "Resistors_ThroughHole:R_Axial_DIN0207_L6.3mm_D2.5mm_P10.16mm_Horizontal" V 5880 4300 50  0001 C CNN
 F 3 "" H 5950 4300 50  0000 C CNN
 	1    5950 4300
@@
 Wire Wire Line
 	1150 2650 1150 3200
-$Comp
-L VDD #PWR04
-U 1 1 5838B631
-P 6900 2450
-F 0 "#PWR04" H 6900 2300 50  0001 C CNN
-F 1 "VDD" H 6900 2600 50  0000 C CNN
-F 2 "" H 6900 2450 50  0000 C CNN
-F 3 "" H 6900 2450 50  0000 C CNN
-	1    6900 2450
-	0    -1   -1   0
-$EndComp
 Wire Wire Line
 	6900 2450 7150 2450
-$Comp
-L VDD #PWR05
-U 1 1 5838BC10
-P 1150 3200
-F 0 "#PWR05" H 1150 3050 50  0001 C CNN
-F 1 "VDD" H 1150 3350 50  0000 C CNN
-F 2 "" H 1150 3200 50  0000 C CNN
-F 3 "" H 1150 3200 50  0000 C CNN
-	1    1150 3200
-	-1   0    0    1
-$EndComp
 NoConn ~ 1700 1000
 NoConn ~ 1650 1850
@@
 GND
 NoConn ~ 7150 2250
+Text GLabel 6900 2450 0    60   Input ~ 0
+VDD
+Text GLabel 1150 3200 0    60   Input ~ 0
+VDD
 $EndSCHEMATC
